Commit message: Updated template to build in humble

File: snp_automate_2022/urdf/workcell.xacro (robot description, xacro)
@@ -130,5 +130,5 @@
     <child link="ee"/>
   </joint>
-  <xacro:property name="camera_cal" value="${load_yaml('$(find snp_automate_2022)/config/camera_calibration.yaml')}" />
+  <xacro:property name="camera_cal" value="${xacro.load_yaml('$(find snp_automate_2022)/config/camera_calibration.yaml')}" />
   <link name="camera_color_optical_frame"/>
   <joint name="tool0_to_camera" type="fixed">
